File: electrical/eagle/soleful/Soleful.sch (EAGLE design)
At the start: 91 parts, among them IC1 STM32F405RGT, IC3 STM32F405RGT, Q1 8MHz, Q2 32.768kHz, Q3 BSS138, Q4 BSS138, Q5 TSX-3225/26MHz/10PPM/7pF/3.2x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, U1 MCP1802, U3 ESP8266, U4 W25Q16BVSSIG, Y1 32.768kHz

Commit message: Work on schematic, starting from scratch due to lack of updated pyboard eagle files
Parts:
- removed ANT: WIFI_ANT_ESP8266, OLIMEX_ANT:WIFI_ANT_ESP8266
- removed C20: 0.1uF, microbuilder:CAP_CERAMIC0805-NOOUTLINE
- removed C21: 0.1uF, microbuilder:CAP_CERAMIC0805_10MGAP
- removed C24: 5.6pF, rcl:C-EU025-024X044
- removed C25, C28: 100nF, rcl:C-EU025-024X044
- removed C26: 10uF, rcl:C-EU025-024X044
- removed C27: NA, rcl:C-EU025-024X044
- removed C29, C30: 10pF, rcl:C-EU025-024X044
- removed D2: 1n4148, microbuilder:DIODESOD-323
- removed GPIO0, GPIO2, MTDO: Default:Open, jumper:SJ2W
- removed GPIO4, GPIO5: TESTPAD32/56, gogo:TESTPAD32/56
- removed IC3: STM32F405RGT, pyboard:STM32F405RGT
- removed L1, L2: NA, rcl:L-US0204/5
- removed Q3: BSS138, microbuilder:MOSFET-NWIDE
- removed Q5: TSX-3225/26MHz/10PPM/7pF/3.2x2.5mm SMD, OLIMEX_DISCRET:SMALL_SMD_CRYSTAL_1
- removed R28: 12k, rcl:R-EU_0204/2V
- removed R29, R33, R34, R35: 200R, rcl:R-EU_0204/2V
- removed U$9: BNO055, microbuilder:BNO055
- removed U3: ESP8266, OLIMEX_IC:ESP8266
- removed U4: W25Q16BVSSIG, OLIMEX_IC:W25Q16BVSSIG
- removed Y1: 32.768kHz, microbuilder:CRYSTAL8.0X3.8
- added IC2: STM32F405RGT, pyboard:STM32F405RGT
- added JBL, JBR1, JBR2, JBR3, JBR4: 1, pinhead:PINHD-1X1
- added JBOT: 8, pinhead:PINHD-1X8
- added JLEFT: 14, pinhead:PINHD-1X14
- added JPOW: 8, pinhead:PINHD-2X4
- added JRIGHT: 11, pinhead:PINHD-1X11
- C11, C12: value 12p -> 2.2pF; device rcl:C-EUC0603 -> SparkFun-Capacitors:10NF-0603-50V-10%
- C16, C17: value 1u -> 12p
- C18, C19: value 22pF -> 1u; device microbuilder:CAP_CERAMIC0805-NOOUTLINE -> rcl:C-EUC0603
- Q4: value BSS138 -> 32.768kHz; device microbuilder:MOSFET-NWIDE -> pyboard:TXC-CRYSTAL32X15
- R10: value 1k -> 4k7
- R11: value 1k -> 4.7k; device rcl:R-EU_R0603 -> SparkFun-Resistors:4.7KOHM-0603-1/10W-1%
- R12: value 100k -> 4.7k; device rcl:R-EU_R0603 -> SparkFun-Resistors:4.7KOHM-0603-1/10W-1%
- R13: value 10M -> 100k; device rcl:R-EU_R0603 -> SparkFun-Resistors:100KOHM-0603-1/10W-1%
- R14: device rcl:R-EU_R0603 -> SparkFun-Resistors:100KOHM-0603-1/10W-1%
- R15: value 100k -> 4k7
- R16: value 0 -> 1k
- R17: value 10k -> 1k
- R18: value 0 -> 100k; device rcl:R-EU_R0805 -> rcl:R-EU_R0603
- R19: value 10K -> 10M; device microbuilder:RESISTOR0805_NOOUTLINE -> rcl:R-EU_R0603
- R20, R21: value 10K -> 100k; device microbuilder:RESISTOR0805_NOOUTLINE -> SparkFun-Resistors:100KOHM-0603-1/10W-1%
- R22, R23: value 10K -> 100k; device microbuilder:RESISTOR0805_NOOUTLINE -> rcl:R-EU_R0603
- R24: value 10K -> 0; device microbuilder:RESISTOR_0805MP -> rcl:R-EU_R0603
- R25: value 10K -> 10k; device microbuilder:RESISTOR_0805MP -> rcl:R-EU_R0603
- R26: value 10K -> 0; device microbuilder:RESISTOR0805_NOOUTLINE -> rcl:R-EU_R0805
- R8, R9: value 4k7 -> 4.7k; device rcl:R-EU_R0603 -> SparkFun-Resistors:4.7KOHM-0603-1/10W-1%
Connections:
- removed net 5.0V: R24.2, R25.2
- removed net GPIO0: GPIO0.2, R33.1
- removed net GPIO2: GPIO2.2, R34.1
- removed net GPIO4: GPIO4.PP, U3.GPIO4
- removed net GPIO5: GPIO5.PP, U3.GPIO5
- removed net I2CADDR_3V: R21.1, U$9.COM3/I2C_ADDR
- removed net INT_3V: U$9.INT
- removed net MTDO: MTDO.2, R35.1
- removed net N$1: C11B.1, IC1.VCAP_2
- removed net N$17: C20.2, U$9.CAP
- removed net N$18: C24.2, L2.2, U3.LNA
- removed net N$19: ANT.ANT, C24.1, L1.2
- removed net N$2: C12B.1, IC1.VCAP_1
- removed net N$20: C27.1, U3.TOUT
- removed net N$21: C29.2, Q5.2, U3.XTAL_OUT
- removed net N$22: R28.1, U3.RES12K
- removed net N$23: C30.2, Q5.1, U3.XTAL_IN
- removed net N$27: R29.2, U3.SD_CLK
- removed net N$28: R33.2, U3.GPIO0
- removed net N$29: R34.2, U3.GPIO2
- removed net N$30: R35.2, U3.MTDO
- removed net N$5 (its old number): C12.2, IC1.PC14, Q2.P$1
- removed net N$8 (its old number): C18.2, U$9.XIN32, Y1.2
- removed net NRESET_3V: D2.A, R26.1, U$9.NRESET
- removed net PS0_3V: R19.1, U$9.PS0
- removed net PS1_3V: R20.1, U$9.PS1
- removed net RST_5V: D2.C
- removed net SCL_3V: Q4.S, R23.1, U$9.COM1/SCL/RX
- removed net SCL_5V: Q4.D, R25.1
- removed net SDA_3V: Q3.S, R22.1, U$9.COM0/SDA/TX
- removed net SDA_5V: Q3.D, R24.1
- removed net SD_CLK: R29.1, U4.CLK
- removed net SD_CMD: U3.SD_CMD, U4./CS/
- removed net SD_D0: U3.SD_DATA_0, U4.DO/IO1
- removed net SD_D1: U3.SD_DATA_1, U4.DI/IO0
- removed net SD_D2: U3.SD_DATA_2, U4./HOLD/IO3
- removed net SD_D3: U3.SD_DATA_3, U4./WP/IO2
- removed net WIFI_RX: IC1.PA3, U3.U0TXD
- removed net WIFI_TX: IC1.PA2, U3.U0RXD
- new net 3V3: R11.2, R12.2, R13.2, R21.2, R8.2, R9.2
- new net IO_PA2: IC2.PA2, JBR2.1
- new net IO_PA3: IC2.PA3, JBR1.1
- new net N$3: C11B.1, IC2.VCAP_2
- new net N$4: C12B.1, IC2.VCAP_1
- new net N1: C12.1, IC1.PC14, Q4.P$1
- new net N2: C11.1, IC1.PC15, Q4.P$2
- new net PA0-X1: IC1.PA0
- new net PA1-X2: IC1.PA1
- new net PA10-ID: IC1.PA10, R21.1
- new net PA11-DM: IC1.PA11
- new net PA12-DP: IC1.PA12
- new net PA13-RED-P5: IC1.PA13
- new net PA14-GRN-P4: IC1.PA14
- new net PA15-YEL-P3: IC1.PA15
- new net PA2-X3: IC1.PA2
- new net PA3-X4: IC1.PA3
- new net PA4-X5: IC1.PA4
- new net PA5-X6: IC1.PA5
- new net PA6-X7: IC1.PA6
- new net PA7-X8: IC1.PA7
- new net PA8-SDIO_SW: IC1.PA8
- new net PA9-VBUS: IC1.PA9
- new net PB0-Y11: IC1.PB0
- new net PB1-Y12: IC1.PB1
- new net PB10-Y9: IC1.PB10, R11.1
- new net PB11-Y10: IC1.PB11, R12.1
- new net PB12-Y5: IC1.PB12
- new net PB13-Y6: IC1.PB13
- new net PB14-Y7: IC1.PB14
- new net PB15-Y8: IC1.PB15
- new net PB2-BOOT1-MMA-INT: IC1.PB2, R14.2
- new net PB3-SW-X17: IC1.PB3
- new net PB4-BLU-P2: IC1.PB4
- new net PB5-MMA_AVDD: IC1.PB5, R20.2
- new net PB6-SCL-X9: IC1.PB6, R9.1
- new net PB7-SDA-X10: IC1.PB7, R8.1
- new net PB8-Y3: IC1.PB8
- new net PB9-Y4: IC1.PB9
- new net PC0-X19: IC1.PC0
- new net PC1-X20: IC1.PC1
- new net PC10-SDIO_D2: IC1.PC10
- new net PC11-SDIO_D3: IC1.PC11, R13.1
- new net PC12-SDIO_CK: IC1.PC12
- new net PC13-X18: IC1.PC13
- new net PC2-X21: IC1.PC2
- new net PC3-X22: IC1.PC3
- new net PC4-X11: IC1.PC4
- new net PC5-X12: IC1.PC5
- new net PC6-Y1: IC1.PC6
- new net PC7-Y2: IC1.PC7
- new net PC8-SDIO_D0: IC1.PC8
- new net PC9-SDIO_D1: IC1.PC9
- new net PD2-SDIO_CMD: IC1.PD2
- net +3V3: now also C19.1, IC2.VBAT, IC2.VDD@19, IC2.VDD@32, IC2.VDD@48, IC2.VDD@64, IC2.VDDA, JBL.1, JLEFT.1, R10.1, R15.1; no longer C17.1, C21.2, C25.1, C26.1, C28.1, GPIO0.1, GPIO2.1, IC1.VBAT, IC1.VDD@19, IC1.VDD@32, IC1.VDD@48, IC1.VDD@64, IC1.VDDA, MTDO.1, Q3.G, Q4.G, R22.2, R23.2, R26.2, R8.1, R9.1, U$9.NBOOT_LOAD_PIN, U$9.VDD, U$9.VDDIO, U3.CHIP_EN, U3.EXT_RSTB, U3.VDD3P3, U3.VDD3P3@1, U3.VDDA, U3.VDDA@1, U3.VDDD, U3.VDDPST, U3.VDDPST@1, U4.VCC
- net BOOT0: now also IC2.BOOT0, JBOT.1, R23.1; no longer IC1.BOOT0, R15.1
- net FS_DM: now also IC2.PA11; no longer IC1.PA11
- net FS_DP: now also IC2.PA12; no longer IC1.PA12
- net FS_VUSB: now also IC2.PA9, R16.2; no longer IC1.PA9, R10.2
- net GND: now also C11.2, C12.2, C16.1, C17.1, C18.2, C19.2, IC2.VSS@18, IC2.VSS@63, IC2.VSSA, JLEFT.2, JPOW.1, JPOW.3, JPOW.5, JPOW.7, JRIGHT.2, R14.1, R17.2, R18.2, R20.1, R22.2, R23.2; no longer ANT.GND, C11.1, C12.1, C16.2, C17.2, C18.1, C19.1, C20.1, C21.1, C25.2, C26.2, C27.2, C28.2, C29.1, C30.1, GPIO0.3, GPIO2.3, IC1.VSS@18, IC1.VSS@63, IC1.VSSA, L1.1, L2.1, MTDO.3, Q5.GND, Q5.GND@1, R11.2, R12.2, R13.2, R14.2, R15.2, R20.2, R21.2, R28.2, U$9.COM2(GND), U$9.GND@1, U$9.GND@2, U$9.PIN10(GND), U$9.PIN15(GND), U$9.PIN16(GND), U3.GND, U3.GND@1, U3.GND@2, U3.GND@3, U3.GND@4, U3.GND@5, U3.GND@6, U3.GND@7, U3.GND@8, U3.GND@9, U4.GND
- net IO_PA0: now also IC2.PA0, JBR4.1; no longer IC1.PA0
- net IO_PA1: now also IC2.PA1, JBR3.1; no longer IC1.PA1
- net IO_PA14: now also IC2.PA14, JLEFT.9; no longer IC1.PA14
- net IO_PA15: now also IC2.PA15, JLEFT.10; no longer IC1.PA15
- net IO_PA4: now also IC2.PA4, JRIGHT.11; no longer IC1.PA4
- net IO_PA5: now also IC2.PA5, JRIGHT.10; no longer IC1.PA5
- net IO_PA6: now also IC2.PA6, JRIGHT.9; no longer IC1.PA6
- net IO_PA7: now also IC2.PA7, JRIGHT.8; no longer IC1.PA7
- net IO_PB0: now also IC2.PB0, JRIGHT.7; no longer IC1.PB0
- net IO_PB1: now also IC2.PB1, JRIGHT.6; no longer IC1.PB1
- net IO_PB10: now also IC2.PB10, JRIGHT.5; no longer IC1.PB10
- net IO_PB11: now also IC2.PB11, JRIGHT.4, R18.1; no longer IC1.PB11, R12.1
- net IO_PB12: now also IC2.PB12, JRIGHT.3; no longer IC1.PB12
- net IO_PB13: now also IC2.PB13, JLEFT.3; no longer IC1.PB13
- net IO_PB14: now also IC2.PB14, JLEFT.4; no longer IC1.PB14
- net IO_PB15: now also IC2.PB15, JLEFT.5; no longer IC1.PB15
- net IO_PB2: now also IC2.PB2, R17.1; no longer IC1.PB2, R11.1
- net IO_PB3: now also IC2.PB3, JLEFT.11; no longer IC1.PB3
- net IO_PB4: now also IC2.PB4, JLEFT.12; no longer IC1.PB4
- net IO_PB9: now also IC2.PB9, JBOT.4; no longer IC1.PB9
- net IO_PC0: now also IC2.PC0, JBOT.5; no longer IC1.PC0
- net IO_PC1: now also IC2.PC1, JBOT.6; no longer IC1.PC1
- net IO_PC2: now also IC2.PC2, JBOT.7; no longer IC1.PC2
- net IO_PC3: now also IC2.PC3, JBOT.8; no longer IC1.PC3
- net IO_PC6: now also IC2.PC6, JLEFT.6; no longer IC1.PC6
- net IO_PC7: now also IC2.PC7, JLEFT.7; no longer IC1.PC7
- net LEDG1: now also IC2.PC4; no longer IC1.PC4
- net LEDG2: now also IC2.PC5; no longer IC1.PC5
- net LEDR1: now also IC2.PA8; no longer IC1.PA8
- net LEDR2: now also IC2.PA10, R24.2; no longer IC1.PA10, R16.2
- net MMA_AVDD: now also IC2.PB5, R22.1; no longer IC1.PB5, R14.1
- net MMA_INT: now also IC2.PB8, JBOT.3; no longer IC1.PB8
- net MMA_SCL: now also IC2.PB6, JLEFT.13, R15.2; no longer IC1.PB6, R9.2
- net MMA_SDA: now also IC2.PB7, JLEFT.14, R10.2; no longer IC1.PB7, R8.2
- net N$10: now also IC2.PH0; no longer IC1.PH0
- net N$15: now also R24.1, U$7.ID; no longer R17.2, U$3.1@A, U$3.1@B
- net N$16: now also R25.2, U$3.1@A, U$3.1@B; no longer C19.2, U$9.XOUT32, Y1.1
- net N$6: now also C17.2, IC2.PC14, Q2.P$1; no longer C11.2, IC1.PC15, Q2.P$2
- net N$7: now also C16.2, IC2.PC15, Q2.P$2; no longer R16.1, U$7.ID
- net N$9: now also IC2.PH1; no longer IC1.PH1
- net NRST: now also IC2.NRST, JBOT.2; no longer IC1.NRST
- net SDIO_CK: now also IC2.PC12; no longer IC1.PC12
- net SDIO_CMD: now also IC2.PD2; no longer IC1.PD2
- net SDIO_D0: now also IC2.PC8; no longer IC1.PC8
- net SDIO_D1: now also IC2.PC9; no longer IC1.PC9
- net SDIO_D2: now also IC2.PC10; no longer IC1.PC10
- net SDIO_D3: now also IC2.PC11, R19.1; no longer IC1.PC11, R13.1
- net SDIO_SW: now also IC2.PC13; no longer IC1.PC13
- net USR_SW: now also IC2.PA13, JLEFT.8, R25.1; no longer IC1.PA13, R17.1
- net VIN: now also C18.1, JPOW.2, JPOW.4, JPOW.6, JPOW.8, JRIGHT.1, R26.1; no longer C16.1, R18.1
- net VUSB: now also R16.1, R26.2; no longer R10.1, R18.2
Other:
- note added: "I2C Pullups"
- note added: "USB"
- note added: "uSD"
- note removed: "0"
- note removed: "1"
- note removed: "FLASH"
- note removed: "GPIO0"
- note removed: "GPIO2"
- note removed: "MOD-WIFI-ESP8266, board revision A"
- note removed: "MTDO"
- note removed: "SDIO"
- note removed: "UART"
- note removed: "X"

Commit message: Finished IC-related wiring
Parts:
- removed C11B, C12B: 2u2, rcl:C-EUC0603
- removed C14, C15: 100n, rcl:C-EUC0603
- removed C16, C17: 12p, rcl:C-EUC0603
- removed C18: 1u, rcl:C-EUC0603
- removed D1: 1N5819, pyboard:1N5819
- removed IC2: STM32F405RGT, pyboard:STM32F405RGT
- removed JBL, JBR1, JBR2, JBR3, JBR4: 1, pinhead:PINHD-1X1
- removed JBOT: 8, pinhead:PINHD-1X8
- removed JLEFT: 14, pinhead:PINHD-1X14
- removed JPOW: 8, pinhead:PINHD-2X4
- removed JRIGHT: 11, pinhead:PINHD-1X11
- removed Q1: 8MHz, pyboard:TXC-CRYSTAL50X32
- removed Q2: 32.768kHz, pyboard:TXC-CRYSTAL32X15
- removed R1, R2: 22, rcl:R-EU_R0603
- removed R10: 4k7, rcl:R-EU_R0603
- removed R16, R17: 1k, rcl:R-EU_R0603
- removed R18, R22, R23: 100k, rcl:R-EU_R0603
- removed R19: 10M, rcl:R-EU_R0603
- removed R24: 0, rcl:R-EU_R0603
- removed R25: 10k, rcl:R-EU_R0603
- removed R26: 0, rcl:R-EU_R0805
- removed R4, R5, R6, R7: 560, rcl:R-EU_R0603
- removed U$1, U$6: LTST-C195KGJRKT, pyboard:LTST-C195KGJRKT
- removed U$2, U$3: KMR4TACTILE, pyboard:KMR4TACTILE
- removed U$4: MOLEX-SD-105027, pyboard:MOLEX-SD-105027
- removed U$5: MMA7660, pyboard:MMA7660
- removed U$7: USB-MICRO-AB, pyboard:USB-MICRO-AB
- removed U1: MCP1802, pyboard:MCP1802
- added C20: 2.2uF, SparkFun-Retired:2.2UF-CERCAP-07888
- added L1: 27uH, SparkFun-Coils:INDUCTOR-SDR13-27UH
- added SW1: RST, SparkFun-Switches:MOMENTARY-SWITCH-SPST-2-SMD-4.6X2.8MM
- added Y1: 12 MHz, crystal:FA-128
- C1, C2: value 12p -> 10pF; device rcl:C-EUC0603 -> SparkFun-Capacitors:10PF-0603-50V-5%
- C10: value 1u -> 4.7uF; device rcl:C-EUC0603 -> SparkFun-Capacitors:4.7UF0603
- C13, C3, C4, C5, C6, C8, C9: value 100n -> 100nF; device rcl:C-EUC0603 -> SparkFun-Capacitors:10NF-0603-50V-10%
- C19: value 1u -> 2.2uF; device rcl:C-EUC0603 -> SparkFun-Retired:2.2UF-CERCAP-07888
- C7: value 4u7 -> 4.7uF; device rcl:C-EUC0603 -> SparkFun-Capacitors:4.7UF0603
- R15: value 4k7 -> 100k; device rcl:R-EU_R0603 -> SparkFun-Resistors:100KOHM-0603-1/10W-1%
- R3: value 10k -> 4.7k; device rcl:R-EU_R0603 -> SparkFun-Resistors:4.7KOHM-0603-1/10W-1%
Connections:
- removed net +3V3: C10.1, C14.1, C19.1, C3.1, C4.1, C5.1, C6.1, C7.1, C8.1, C9.1, IC2.VBAT, IC2.VDD@19, IC2.VDD@32, IC2.VDD@48, IC2.VDD@64, IC2.VDDA, JBL.1, JLEFT.1, R10.1, R15.1, R3.1, U$1.A1, U$1.A2, U$4.VDD, U$5.DVDD, U$6.A1, U$6.A2, U1.VOUT
- removed net BOOT0: IC2.BOOT0, JBOT.1, R23.1
- removed net FS_DM: IC2.PA11, R1.2
- removed net FS_DP: IC2.PA12, R2.2
- removed net FS_VUSB: IC2.PA9, R16.2
- removed net IO_PA0: IC2.PA0, JBR4.1
- removed net IO_PA1: IC2.PA1, JBR3.1
- removed net IO_PA14: IC2.PA14, JLEFT.9
- removed net IO_PA15: IC2.PA15, JLEFT.10
- removed net IO_PA2: IC2.PA2, JBR2.1
- removed net IO_PA3: IC2.PA3, JBR1.1
- removed net IO_PA4: IC2.PA4, JRIGHT.11
- removed net IO_PA5: IC2.PA5, JRIGHT.10
- removed net IO_PA6: IC2.PA6, JRIGHT.9
- removed net IO_PA7: IC2.PA7, JRIGHT.8
- removed net IO_PB0: IC2.PB0, JRIGHT.7
- removed net IO_PB1: IC2.PB1, JRIGHT.6
- removed net IO_PB10: IC2.PB10, JRIGHT.5
- removed net IO_PB11: IC2.PB11, JRIGHT.4, R18.1
- removed net IO_PB12: IC2.PB12, JRIGHT.3
- removed net IO_PB13: IC2.PB13, JLEFT.3
- removed net IO_PB14: IC2.PB14, JLEFT.4
- removed net IO_PB15: IC2.PB15, JLEFT.5
- removed net IO_PB2: IC2.PB2, R17.1
- removed net IO_PB3: IC2.PB3, JLEFT.11
- removed net IO_PB4: IC2.PB4, JLEFT.12
- removed net IO_PB9: IC2.PB9, JBOT.4
- removed net IO_PC0: IC2.PC0, JBOT.5
- removed net IO_PC1: IC2.PC1, JBOT.6
- removed net IO_PC2: IC2.PC2, JBOT.7
- removed net IO_PC3: IC2.PC3, JBOT.8
- removed net IO_PC6: IC2.PC6, JLEFT.6
- removed net IO_PC7: IC2.PC7, JLEFT.7
- removed net LEDG1: IC2.PC4, R4.1
- removed net LEDG2: IC2.PC5, R7.1
- removed net LEDR1: IC2.PA8, R6.1
- removed net LEDR2: IC2.PA10, R24.2, R5.1
- removed net MMA_AVDD: C15.1, IC2.PB5, R22.1, U$5.AVDD
- removed net MMA_INT: IC2.PB8, JBOT.3, U$5.INT
- removed net MMA_SCL: IC2.PB6, JLEFT.13, R15.2, U$5.SCL
- removed net MMA_SDA: IC2.PB7, JLEFT.14, R10.2, U$5.SDA
- removed net N$10: C2.2, IC2.PH0, Q1.P$1
- removed net N$11: R4.2, U$1.K1
- removed net N$12: R5.2, U$6.K2
- removed net N$13: R6.2, U$1.K2
- removed net N$14: R7.2, U$6.K1
- removed net N$15: R24.1, U$7.ID
- removed net N$16: R25.2, U$3.1@A, U$3.1@B
- removed net N$3: C11B.1, IC2.VCAP_2
- removed net N$4: C12B.1, IC2.VCAP_1
- removed net N$5: R2.1, U$7.D+
- removed net N$6: C17.2, IC2.PC14, Q2.P$1
- removed net N$7: C16.2, IC2.PC15, Q2.P$2
- removed net N$8: R1.1, U$7.D-
- removed net N$9: C1.2, IC2.PH1, Q1.P$2
- removed net NRST: C13.1, IC2.NRST, JBOT.2, R3.2, U$2.1@A, U$2.1@B
- removed net SDIO_CK: IC2.PC12, U$4.CLK
- removed net SDIO_CMD: IC2.PD2, U$4.CMD
- removed net SDIO_D0: IC2.PC8, U$4.DAT0
- removed net SDIO_D1: IC2.PC9, U$4.DAT1
- removed net SDIO_D2: IC2.PC10, U$4.DAT2
- removed net SDIO_D3: IC2.PC11, R19.1, U$4.DAT3
- removed net SDIO_SW: IC2.PC13, U$4.SWITCH
- removed net USR_SW: IC2.PA13, JLEFT.8, R25.1
- removed net VIN: C18.1, D1.K, JPOW.2, JPOW.4, JPOW.6, JPOW.8, JRIGHT.1, R26.1, U1.EN, U1.VIN
- removed net VUSB: D1.A, R16.1, R26.2, U$7.VUSB
- new net A3V3: C10.1, C9.1, IC1.VDDA, L1.2
- new net BOOT0-P1: IC1.BOOT0, R15.2
- new net N3: C2.1, IC1.PH0, Y1.1
- new net N4: C1.1, IC1.PH1, Y1.3
- new net RST#: C13.1, IC1.NRST, R3.1, SW1.1
- new net VBACKUP: C8.1, IC1.VBAT
- new net VCAP1: C19.2, IC1.VCAP_1
- new net VCAP2: C20.2, IC1.VCAP_2
- net 3V3: now also C3.1, C4.1, C5.1, C6.1, C7.1, IC1.VDD@19, IC1.VDD@32, IC1.VDD@48, IC1.VDD@64, L1.1, R3.2
- net GND: now also C1.2, C19.1, C2.2, C20.1, IC1.VSS@18, IC1.VSS@63, IC1.VSSA, R15.1, SW1.4, Y1.2, Y1.4; no longer C1.1, C11B.2, C12B.2, C14.2, C15.2, C16.1, C17.1, C18.2, C19.2, C2.1, IC2.VSS@18, IC2.VSS@63, IC2.VSSA, JLEFT.2, JPOW.1, JPOW.3, JPOW.5, JPOW.7, JRIGHT.2, R17.2, R18.2, R19.2, R22.2, R23.2, U$2.0@A, U$2.0@B, U$3.0@A, U$3.0@B, U$4.VSS, U$5.AVSS, U$5.DVSS, U$5.N/C@10, U$5.N/C@2, U$5.RSRVD, U$7.GND, U1.GND
Other:
- note removed: "Analog"
- note removed: "DFU boot"
- note removed: "MMA"
- note removed: "R16 and R18 are unpopulated. Used for optional USB OTG support."
- note removed: "VBAT"
- note removed: "VDD"

Commit message: Further schematic work
Parts:
- added C14, C16: 4.7uF, SparkFun-Capacitors:4.7UF0603
- added C15: 2.2uF, SparkFun-Retired:2.2UF-CERCAP-07888
- added D2: LED-RED, SparkFun-LED:LED-RED0603
- added D3: LED-GREEN, SparkFun-LED:LED-GREEN0603
- added D4: LED-YELLOW, SparkFun-LED:LED-YELLOW0603
- added D5: LED-BLUE, SparkFun-LED:LED-BLUE0603
- added IC2: MCP1703DB, linear:MCP1703DB
- added R10, R4, R5, R7: 560, rcl:R-EU_R0603
- added U$9: MOLEX-SD-105027, pyboard:MOLEX-SD-105027
Connections:
- new net N$3: IC2.GND
- new net N$4: D3.A, R10.2
- new net N$5: D4.A, R7.2
- new net N$6: D5.A, R5.2
- new net N$7: D2.A, R4.2
- new net V+: C15.1, IC2.VI
- net 3V3: now also C14.1, C16.1, IC2.VO, U$9.VDD
- net GND: now also C14.2, C15.2, C16.2, D2.C, D3.C, D4.C, D5.C, U$9.VSS
- net PA13-RED-P5: now also R4.1
- net PA14-GRN-P4: now also R10.1
- net PA15-YEL-P3: now also R7.1
- net PA8-SDIO_SW: now also U$9.SWITCH
- net PB4-BLU-P2: now also R5.1
- net PC10-SDIO_D2: now also U$9.DAT2
- net PC11-SDIO_D3: now also U$9.DAT3
- net PC12-SDIO_CK: now also U$9.CLK
- net PC8-SDIO_D0: now also U$9.DAT0
- net PC9-SDIO_D1: now also U$9.DAT1
- net PD2-SDIO_CMD: now also U$9.CMD

Commit message: further work
Parts:
- added C11B, C12B: 2u2, rcl:C-EUC0603
- added C17, C18: 4.7uF, SparkFun-Capacitors:4.7UF0603
- added C21, C22, C23, C24, C25, C26, C31, C32, C33: 100n, rcl:C-EUC0603
- added C27, C28, C34, C35: 12p, rcl:C-EUC0603
- added C29, C36, C37: 1u, rcl:C-EUC0603
- added C30: 4u7, rcl:C-EUC0603
- added D1: MSE1PB-M3/89A, PP_Passives:DIODE_MICROSMP
- added D6: 1N5819, pyboard:1N5819
- added IC3: STM32F405RGT, pyboard:STM32F405RGT
- added JBL, JBR1, JBR2, JBR3, JBR4: 1, pinhead:PINHD-1X1
- added JBOT: 8, pinhead:PINHD-1X8
- added JLEFT: 14, pinhead:PINHD-1X14
- added JPOW: 8, pinhead:PINHD-2X4
- added JRIGHT: 11, pinhead:PINHD-1X11
- added Q1: MOSFET-PCHANNEL, User-Submitted:MOSFET-PCHANNEL
- added Q2: 8MHz, pyboard:TXC-CRYSTAL50X32
- added Q3: 32.768kHz, pyboard:TXC-CRYSTAL32X15
- added R1, R19, R2, R22: 22, rcl:R-EU_R0603
- added R16, R24, R25, R26, R27, R6: 560, rcl:R-EU_R0603
- added R17: 4.7k, SparkFun-Resistors:4.7KOHM-0603-1/10W-1%
- added R18: 100k, SparkFun-Resistors:100KOHM-0603-1/10W-1%
- added R23, R37: 10k, rcl:R-EU_R0603
- added R28, R29: 4k7, rcl:R-EU_R0603
- added R30, R31: 1k, rcl:R-EU_R0603
- added R32, R34, R35: 100k, rcl:R-EU_R0603
- added R33: 10M, rcl:R-EU_R0603
- added R36: 0, rcl:R-EU_R0603
- added R38: 0, rcl:R-EU_R0805
- added SW2: USR, SparkFun-Switches:MOMENTARY-SWITCH-SPST-2-SMD-4.6X2.8MM
- added U$1, U$5: MMA7660, pyboard:MMA7660
- added U$10, U$8: USB-MICRO-AB, pyboard:USB-MICRO-AB
- added U$2, U$3: KMR4TACTILE, pyboard:KMR4TACTILE
- added U$4: MOLEX-SD-105027, pyboard:MOLEX-SD-105027
- added U$6, U$7: LTST-C195KGJRKT, pyboard:LTST-C195KGJRKT
- added U1: MCP1802, pyboard:MCP1802
- C14: value 4.7uF -> 100nF; device SparkFun-Capacitors:4.7UF0603 -> SparkFun-Capacitors:10NF-0603-50V-10%
- C15: value 2.2uF -> 100nF; device SparkFun-Retired:2.2UF-CERCAP-07888 -> SparkFun-Capacitors:10NF-0603-50V-10%
- C16: value 4.7uF -> 2.2uF; device SparkFun-Capacitors:4.7UF0603 -> SparkFun-Retired:2.2UF-CERCAP-07888
Connections:
- new net +3V3: C21.1, C22.1, C23.1, C24.1, C25.1, C26.1, C29.1, C30.1, C32.1, C37.1, IC3.VBAT, IC3.VDD@19, IC3.VDD@32, IC3.VDD@48, IC3.VDD@64, IC3.VDDA, JBL.1, JLEFT.1, R23.1, R28.1, R29.1, U$4.VDD, U$5.DVDD, U$6.A1, U$6.A2, U$7.A1, U$7.A2, U1.VOUT
- new net BOOT0: IC3.BOOT0, JBOT.1, R35.1
- new net DM: R1.2, U$10.D-
- new net DP: R2.2, U$10.D+
- new net FS_DM: IC3.PA11, R19.2
- new net FS_DP: IC3.PA12, R22.2
- new net FS_VUSB: IC3.PA9, R30.2
- new net ID: R16.2, U$10.ID
- new net IO_PA0: IC3.PA0, JBR4.1
- new net IO_PA1: IC3.PA1, JBR3.1
- new net IO_PA14: IC3.PA14, JLEFT.9
- new net IO_PA15: IC3.PA15, JLEFT.10
- new net IO_PA2: IC3.PA2, JBR2.1
- new net IO_PA3: IC3.PA3, JBR1.1
- new net IO_PA4: IC3.PA4, JRIGHT.11
- new net IO_PA5: IC3.PA5, JRIGHT.10
- new net IO_PA6: IC3.PA6, JRIGHT.9
- new net IO_PA7: IC3.PA7, JRIGHT.8
- new net IO_PB0: IC3.PB0, JRIGHT.7
- new net IO_PB1: IC3.PB1, JRIGHT.6
- new net IO_PB10: IC3.PB10, JRIGHT.5
- new net IO_PB11: IC3.PB11, JRIGHT.4, R32.1
- new net IO_PB12: IC3.PB12, JRIGHT.3
- new net IO_PB13: IC3.PB13, JLEFT.3
- new net IO_PB14: IC3.PB14, JLEFT.4
- new net IO_PB15: IC3.PB15, JLEFT.5
- new net IO_PB2: IC3.PB2, R31.1
- new net IO_PB3: IC3.PB3, JLEFT.11
- new net IO_PB4: IC3.PB4, JLEFT.12
- new net IO_PB9: IC3.PB9, JBOT.4
- new net IO_PC0: IC3.PC0, JBOT.5
- new net IO_PC1: IC3.PC1, JBOT.6
- new net IO_PC2: IC3.PC2, JBOT.7
- new net IO_PC3: IC3.PC3, JBOT.8
- new net IO_PC6: IC3.PC6, JLEFT.6
- new net IO_PC7: IC3.PC7, JLEFT.7
- new net LEDG1: IC3.PC4, R24.1
- new net LEDG2: IC3.PC5, R27.1
- new net LEDR1: IC3.PA8, R26.1
- new net LEDR2: IC3.PA10, R25.1, R36.2
- new net MMA_AVDD: C33.1, IC3.PB5, R34.1, U$5.AVDD
- new net MMA_INT: IC3.PB8, JBOT.3, U$5.INT
- new net MMA_SCL: IC3.PB6, JLEFT.13, R29.2, U$5.SCL
- new net MMA_SDA: IC3.PB7, JLEFT.14, R28.2, U$5.SDA
- new net N$10: Q1.D
- new net N$11: C12B.1, IC3.VCAP_1
- new net N$12: R22.1, U$8.D+
- new net N$13: C28.2, IC3.PH0, Q2.P$1
- new net N$14: R24.2, U$6.K1
- new net N$15: R25.2, U$7.K2
- new net N$16: R26.2, U$6.K2
- new net N$17: C35.2, IC3.PC14, Q3.P$1
- new net N$18: C34.2, IC3.PC15, Q3.P$2
- new net N$19: C27.2, IC3.PH1, Q2.P$2
- new net N$20: R27.2, U$7.K1
- new net N$21: R19.1, U$8.D-
- new net N$22: R36.1, U$8.ID
- new net N$23: R37.2, U$3.1@A, U$3.1@B
- new net N$8: D1.ANODE, Q1.G, R10.2, R18.2, U$10.VUSB
- new net N$9: C11B.1, IC3.VCAP_2
- new net NRST: C31.1, IC3.NRST, JBOT.2, R23.2, U$2.1@A, U$2.1@B
- new net SDIO_CK: IC3.PC12, U$4.CLK
- new net SDIO_CMD: IC3.PD2, U$4.CMD
- new net SDIO_D0: IC3.PC8, U$4.DAT0
- new net SDIO_D1: IC3.PC9, U$4.DAT1
- new net SDIO_D2: IC3.PC10, U$4.DAT2
- new net SDIO_D3: IC3.PC11, R33.1, U$4.DAT3
- new net SDIO_SW: IC3.PC13, U$4.SWITCH
- new net USR-SW: R17.1, SW2.3
- new net USR_SW: IC3.PA13, JLEFT.8, R37.1
- new net VIN: C36.1, D6.K, JPOW.2, JPOW.4, JPOW.6, JPOW.8, JRIGHT.1, R38.1, U1.EN, U1.VIN
- new net VUSB: D6.A, R30.1, R38.2, U$8.VUSB
- net 3V3: now also C17.1, C18.1, D1.CATHODE, Q1.S, U$1.DVDD; no longer C16.1
- net GND: now also C11B.2, C12B.2, C17.2, C18.2, C21.2, C22.2, C23.2, C24.2, C25.2, C26.2, C27.1, C28.1, C29.2, C30.2, C31.2, C32.2, C33.2, C34.1, C35.1, C36.2, C37.2, IC3.VSS@18, IC3.VSS@63, IC3.VSSA, JLEFT.2, JPOW.1, JPOW.3, JPOW.5, JPOW.7, JRIGHT.2, R18.1, R31.2, R32.2, R33.2, R34.2, R35.2, SW2.1, U$1.AVSS, U$1.DVSS, U$1.N/C@10, U$1.N/C@2, U$1.RSRVD, U$10.GND, U$2.0@A, U$2.0@B, U$3.0@A, U$3.0@B, U$4.VSS, U$5.AVSS, U$5.DVSS, U$5.N/C@10, U$5.N/C@2, U$5.RSRVD, U$8.GND, U1.GND
- net N$4: now also R6.2; no longer R10.2
- net PA10-ID: now also R16.1
- net PA11-DM: now also R1.1
- net PA12-DP: now also R2.1
- net PA14-GRN-P4: now also R6.1; no longer R10.1
- net PA9-VBUS: now also R10.1
- net PB2-BOOT1-MMA-INT: now also U$1.INT
- net PB3-SW-X17: now also R17.2
- net PB5-MMA_AVDD: now also C15.1, U$1.AVDD
- net PB6-SCL-X9: now also U$1.SCL
- net PB7-SDA-X10: now also U$1.SDA
- net V+: now also C16.1; no longer C15.1
Other:
- note added: "Analog"
- note added: "DFU boot"
- note added: "Jeet Mehta"
- note added: "MMA"
- note added: "R16 and R18 are unpopulated. Used for optional USB OTG support."
- note added: "VBAT"
- note added: "VDD"
